File: SOP24/MBI5030-SOP24_starter-board__panel.kicad_pcb (KiCad board)
At the start: 2 copper layers, 97.1 x 99.4 mm, 546 parts, among them IC1 MBI5030GF, P3 CONN_12, P4 CONN_12

Commit message: Upgraded the panel as well.
Parts:
- removed R1 (x12), R10 (x12), R11 (x12), R12 (x12), R13 (x12), R14 (x12), R15 (x12), R16 (x12), R2 (x12), R3 (x12), R4 (x12), R5 (x12), R6 (x12), R7 (x12), R8 (x12), R9 (x12): 1k, MADW__R0603
- removed the R17 at (122.1, 145.5)
- removed the R17 at (154.8, 70.2)
- removed the R17 at (154.8, 120.4)
- removed the R17 at (154.8, 145.5)
- removed the R17 at (122.1, 120.4)
- removed the R17 at (122.1, 70.2)
- removed the R17 at (122.1, 95.3)
- removed the R17 at (89.4, 95.3)
- removed the R17 at (89.4, 70.2)
- removed the R17 at (89.4, 120.4)
- removed the R17 at (89.4, 145.5)
- removed the R17 at (154.8, 95.3)
- removed the RV1 at (127.0, 145.8)
- removed the RV1 at (159.7, 70.5)
- removed the RV1 at (159.7, 120.7)
- removed the RV1 at (159.7, 145.8)
- removed the RV1 at (127.0, 120.7)
- removed the RV1 at (127.0, 70.5)
- removed the RV1 at (127.0, 95.6)
- removed the RV1 at (94.3, 95.6)
- removed the RV1 at (94.3, 70.5)
- removed the RV1 at (94.3, 120.7)
- removed the RV1 at (94.3, 145.8)
- removed the RV1 at (159.7, 95.6)
- added R17: 300R, MADW__R0603, F.Cu at (89.4, 70.2)
- added R17: 300R, MADW__R0603, F.Cu at (154.8, 95.2)
- added R17: 300R, MADW__R0603, F.Cu at (154.8, 120.3)
- added R17: 300R, MADW__R0603, F.Cu at (154.8, 145.4)
- added R17: 300R, MADW__R0603, F.Cu at (89.4, 95.2)
- added R17: 300R, MADW__R0603, F.Cu at (89.4, 120.3)
- added R17: 300R, MADW__R0603, F.Cu at (89.4, 145.4)
- added R17: 300R, MADW__R0603, F.Cu at (122.1, 145.4)
- added R17: 300R, MADW__R0603, F.Cu at (122.1, 120.3)
- added R17: 300R, MADW__R0603, F.Cu at (122.1, 95.2)
- added R17: 300R, MADW__R0603, F.Cu at (122.1, 70.2)
- added R17: 300R, MADW__R0603, F.Cu at (154.8, 70.2)
- added RP1: 1k, MADW__1206*4_resistor_array, F.Cu at (90.5, 73.6)
- added RP1: 1k, MADW__1206*4_resistor_array, F.Cu at (155.8, 98.7)
- added RP1: 1k, MADW__1206*4_resistor_array, F.Cu at (155.8, 123.8)
- added RP1: 1k, MADW__1206*4_resistor_array, F.Cu at (155.8, 148.9)
- added RP1: 1k, MADW__1206*4_resistor_array, F.Cu at (90.5, 98.7)
- added RP1: 1k, MADW__1206*4_resistor_array, F.Cu at (90.5, 123.8)
- added RP1: 1k, MADW__1206*4_resistor_array, F.Cu at (90.5, 148.9)
- added RP1: 1k, MADW__1206*4_resistor_array, F.Cu at (123.2, 148.9)
- added RP1: 1k, MADW__1206*4_resistor_array, F.Cu at (123.2, 123.8)
- added RP1: 1k, MADW__1206*4_resistor_array, F.Cu at (123.2, 98.7)
- added RP1: 1k, MADW__1206*4_resistor_array, F.Cu at (123.2, 73.6)
- added RP1: 1k, MADW__1206*4_resistor_array, F.Cu at (155.8, 73.6)
- added RP2: 1k, MADW__1206*4_resistor_array, F.Cu at (94.3, 74.7)
- added RP2: 1k, MADW__1206*4_resistor_array, F.Cu at (159.8, 99.8)
- added RP2: 1k, MADW__1206*4_resistor_array, F.Cu at (159.8, 124.8)
- added RP2: 1k, MADW__1206*4_resistor_array, F.Cu at (159.8, 149.9)
- added RP2: 1k, MADW__1206*4_resistor_array, F.Cu at (94.3, 99.8)
- added RP2: 1k, MADW__1206*4_resistor_array, F.Cu at (94.3, 124.8)
- added RP2: 1k, MADW__1206*4_resistor_array, F.Cu at (94.3, 149.9)
- added RP2: 1k, MADW__1206*4_resistor_array, F.Cu at (127.0, 149.9)
- added RP2: 1k, MADW__1206*4_resistor_array, F.Cu at (127.0, 124.8)
- added RP2: 1k, MADW__1206*4_resistor_array, F.Cu at (127.0, 99.8)
- added RP2: 1k, MADW__1206*4_resistor_array, F.Cu at (127.0, 74.7)
- added RP2: 1k, MADW__1206*4_resistor_array, F.Cu at (159.8, 74.7)
- added RP3: 1k, MADW__1206*4_resistor_array, F.Cu at (94.3, 65.8)
- added RP3: 1k, MADW__1206*4_resistor_array, F.Cu at (159.8, 90.8)
- added RP3: 1k, MADW__1206*4_resistor_array, F.Cu at (159.8, 116.0)
- added RP3: 1k, MADW__1206*4_resistor_array, F.Cu at (159.8, 141.1)
- added RP3: 1k, MADW__1206*4_resistor_array, F.Cu at (94.3, 90.8)
- added RP3: 1k, MADW__1206*4_resistor_array, F.Cu at (94.3, 116.0)
- added RP3: 1k, MADW__1206*4_resistor_array, F.Cu at (94.3, 141.1)
- added RP3: 1k, MADW__1206*4_resistor_array, F.Cu at (127.0, 141.1)
- added RP3: 1k, MADW__1206*4_resistor_array, F.Cu at (127.0, 116.0)
- added RP3: 1k, MADW__1206*4_resistor_array, F.Cu at (127.0, 90.8)
- added RP3: 1k, MADW__1206*4_resistor_array, F.Cu at (127.0, 65.8)
- added RP3: 1k, MADW__1206*4_resistor_array, F.Cu at (159.8, 65.8)
- added RP4: 1k, MADW__1206*4_resistor_array, F.Cu at (90.5, 67.1)
- added RP4: 1k, MADW__1206*4_resistor_array, F.Cu at (155.8, 92.2)
- added RP4: 1k, MADW__1206*4_resistor_array, F.Cu at (155.8, 117.3)
- added RP4: 1k, MADW__1206*4_resistor_array, F.Cu at (155.8, 142.4)
- added RP4: 1k, MADW__1206*4_resistor_array, F.Cu at (90.5, 92.2)
- added RP4: 1k, MADW__1206*4_resistor_array, F.Cu at (90.5, 117.3)
- added RP4: 1k, MADW__1206*4_resistor_array, F.Cu at (90.5, 142.4)
- added RP4: 1k, MADW__1206*4_resistor_array, F.Cu at (123.2, 142.4)
- added RP4: 1k, MADW__1206*4_resistor_array, F.Cu at (123.2, 117.3)
- added RP4: 1k, MADW__1206*4_resistor_array, F.Cu at (123.2, 92.2)
- added RP4: 1k, MADW__1206*4_resistor_array, F.Cu at (123.2, 67.1)
- added RP4: 1k, MADW__1206*4_resistor_array, F.Cu at (155.8, 67.1)
- added RV1: 2k, MADW__TC33X-POT, F.Cu at (94.3, 70.3)
- added RV1: 2k, MADW__TC33X-POT, F.Cu at (159.8, 95.4)
- added RV1: 2k, MADW__TC33X-POT, F.Cu at (159.8, 120.5)
- added RV1: 2k, MADW__TC33X-POT, F.Cu at (159.8, 145.6)
- added RV1: 2k, MADW__TC33X-POT, F.Cu at (94.3, 95.4)
- added RV1: 2k, MADW__TC33X-POT, F.Cu at (94.3, 120.5)
- added RV1: 2k, MADW__TC33X-POT, F.Cu at (94.3, 145.6)
- added RV1: 2k, MADW__TC33X-POT, F.Cu at (127.0, 145.6)
- added RV1: 2k, MADW__TC33X-POT, F.Cu at (127.0, 120.5)
- added RV1: 2k, MADW__TC33X-POT, F.Cu at (127.0, 95.4)
- added RV1: 2k, MADW__TC33X-POT, F.Cu at (127.0, 70.3)
- added RV1: 2k, MADW__TC33X-POT, F.Cu at (159.8, 70.3)
Connections:
- net N-0000010 renamed /L3A
- net N-0000011 renamed /L4A
- net N-0000012 renamed /L5A
- net N-0000013 renamed /L6A
- net N-0000014 renamed /L7A
- net N-0000015 renamed /L8A
- net N-0000016 renamed /L3B
- net N-0000017 renamed /L5B
- net N-0000019 renamed /L7B
- net N-0000020 renamed /L8B
- net N-000005 renamed /L1B
- net N-000006 renamed /L2B
- net N-000007 renamed /L4B
- net N-000008 renamed /L1A
- net N-000009 renamed /L2A
- D14 pad 1: N-0000018 (its old number) -> /L6B (x12)
Routing:
- net N-0000018: track 896.3 -> 510.9 mm
- net /L8B: track 19.8 -> 172.0 mm
- net /L1A: track 19.8 -> 170.0 mm
- net /L7B: track 19.8 -> 149.4 mm
- net /L2A: track 19.8 -> 146.7 mm
- net /L6B: track 0.00 -> 126.2 mm
- net /L3A: track 19.8 -> 125.5 mm
- net /L5B: track 19.8 -> 103.9 mm
- net /L4A: track 19.8 -> 100.5 mm
- net N-000004: track 64.3 -> 0.00 mm
- net /L4B: track 19.8 -> 75.0 mm
- net /L5A: track 19.8 -> 74.8 mm
- net N-000001: track 0.00 -> 51.2 mm
- net /L3B: track 19.8 -> 61.9 mm
- net /L6A: track 19.8 -> 58.0 mm
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Other:
- board text added: "MBI5030-SOP24_starter-board V1.1 2013 - blog.spitzenpfeil.org"
- board text added: "mA"
- board text removed: "I_SET"
- board text removed: "MBI5030-SOP24_starter-board V1.02 2013 - blog.spitzenpfeil.org"

Commit message: Flipped one trace to F_Cu.
Routing:
- net VCC: vias 12 -> 1
Other:
- net class Default: clearance 0.3 -> 0.15
- rule trace_clearance: 0.3 -> 0.15
- rule trace_min: 0.254 -> 0.15
